Commit message: 有点撞墙但是还行

File: src/urdf_gazebo_demo/xacro/my_laser.urdf.xacro (robot description, xacro)
@@ -51,5 +51,5 @@
             </geometry>
             <origin xyz="0.0 0.0 0.0" rpy="0.0 0.0 0.0" />
-            <material name="Black" />
+            <material name="red" />
         </visual>
         <collision>
